Commit message: Trying to make control work

File: description/robot.urdf.xacro (robot description, xacro)
@@ -1,4 +1,5 @@
 <?xml version="1.0"?>
 <robot xmlns:xacro="http://ros.org/wiki/xacro" name="my_create3">
-  <xacro:include filename="$(find irobot_create_description)/urdf/create3.urdf.xacro" />
+  <xacro:include filename="$(find irobot_create_description)/urdf/create3.urdf.xacro"/>
+  <xacro:include filename="ros2_control.urdf.xacro" />
 </robot>

File: description/ros2_control.urdf.xacro (robot description, xacro)
@@ -5,5 +5,5 @@
       <plugin>gz_ros2_control/GazeboSimSystem</plugin>
     </hardware>
-    <join name="left_wheel">
+    <joint name="left_wheel_joint">
       <command_interface name="velocity">
         <paramp name="min">-10</paramp>
@@ -13,5 +13,5 @@
       <state_interface name="velocity"/>
     </joint>
-    <join name="right_wheel">
+    <joint name="right_wheel_joint">
       <command_interface name="velocity">
         <paramp name="min">-10</paramp>

Commit message: Using irobot_create_control controllers. The robot finally moves

File: description/robot.urdf.xacro (robot description, xacro)
@@ -2,4 +2,3 @@
 <robot xmlns:xacro="http://ros.org/wiki/xacro" name="my_create3">
   <xacro:include filename="$(find irobot_create_description)/urdf/create3.urdf.xacro"/>
-  <xacro:include filename="ros2_control.urdf.xacro" />
 </robot>

File: description/ros2_control.urdf.xacro (robot description, xacro)
@@ -1,29 +1,8 @@
 <?xml version="1.0"?>
-  <robot xmlns:xacro="http://ros.org/wiki/xacro">
-  <ros2_control name="GazeboSystem" type="system">
-    <hardware>
-      <plugin>gz_ros2_control/GazeboSimSystem</plugin>
-    </hardware>
-    <joint name="left_wheel_joint">
-      <command_interface name="velocity">
-        <paramp name="min">-10</paramp>
-        <paramp name="max">10</paramp>
-      </command_interface>
-      <state_interface name="position"/>
-      <state_interface name="velocity"/>
-    </joint>
-    <joint name="right_wheel_joint">
-      <command_interface name="velocity">
-        <paramp name="min">-10</paramp>
-        <paramp name="max">10</paramp>
-      </command_interface>
-      <state_interface name="position"/>
-      <state_interface name="velocity"/>
-    </joint>
-  </ros2_control>
+<robot xmlns:xacro="http://ros.org/wiki/xacro">
   <gazebo>
-     <plugin name="gz_ros2_control::GazeboSimROS2ControlPlugin" filename="libgz_ros2_control-system.so">
-        <parameters>$(find vector-field-simul)/config/controllers.yaml</parameters>
-     </plugin>
+    <plugin name="gz_ros2_control::GazeboSimROS2ControlPlugin" filename="libgz_ros2_control-system.so">
+      <parameters>$(find vector-field-simul)/config/controllers.yaml</parameters>
+    </plugin>
   </gazebo>
-  </robot>
+</robot>
